Commit message: urdf file rename

File: kuka_bringup/urdf/kuka_iiwa.urdf (robot description, URDF)
Before this commit: robot kuka, 19 links, 18 joints
Joints:
- joint back_left_wheel_joint: type continuous -> fixed
- joint back_right_wheel_joint: type continuous -> fixed
- joint front_left_wheel_joint: type continuous -> fixed
- joint front_right_wheel_joint: type continuous -> fixed
- joint joint_a1: type revolute -> fixed
- joint joint_a2: type revolute -> fixed
- joint joint_a3: type revolute -> fixed
- joint joint_a4: type revolute -> fixed
- joint joint_a5: type revolute -> fixed
- joint joint_a6: type revolute -> fixed
- joint joint_a7: type revolute -> fixed

Commit message: small error in joint pose

File: kuka_bringup/urdf/kuka_iiwa.urdf (robot description, URDF)
Before this commit: robot kuka, 19 links, 18 joints
Joints:
- joint laser_B1_joint: origin xyz=0.483 -0.258 -0.112 rpy=0 0 0 -> xyz=0.483 -0.258 -0.112 rpy=0 0 -0.7854
- joint laser_B4_joint: origin xyz=-0.483 0.258 -0.112 rpy=0 0 0 -> xyz=-0.483 0.258 -0.112 rpy=0 0 2.3562
