Commit message: support for using moveit with iiwa manipulator

File: kuka_bringup/urdf/kuka_withD435.urdf (robot description, URDF)
Before this commit: robot kuka, 20 links, 19 joints
Joints:
- joint joint_a1: type fixed -> revolute
- joint joint_a2: type fixed -> revolute
- joint joint_a3: type fixed -> revolute
- joint joint_a4: type fixed -> revolute
- joint joint_a5: type fixed -> revolute
- joint joint_a6: type fixed -> revolute
- joint joint_a7: type fixed -> revolute

Commit message: gripper tool added to urdf

File: kuka_bringup/urdf/kuka_withD435.urdf (robot description, URDF)
Before this commit: robot kuka, 20 links, 19 joints
Links:
- added link gripper_base_link; collision mesh filename=package://kuka_bringup/meshes/gripper/collision/robotiq_arg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; visual mesh filename=package://kuka_bringup/meshes/gripper/visual/robotiq_arg2f_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 scale=0.001 0.001 0.001
- added link left_inner_finger; collision mesh filename=package://kuka_bringup/meshes/gripper/collision/robotiq_arg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 scale=0.001 0.001 0.001; visual mesh filename=package://kuka_bringup/meshes/gripper/visual/robotiq_arg2f_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 scale=0.001 0.001 0.001
- added link left_inner_finger_pad; collision box size=0.022 0.00635 0.0375; visual box size=0.022 0.00635 0.0375
- added link left_inner_knuckle; collision mesh filename=package://kuka_bringup/meshes/gripper/collision/robotiq_arg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 scale=0.001 0.001 0.001; visual mesh filename=package://kuka_bringup/meshes/gripper/visual/robotiq_arg2f_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 scale=0.001 0.001 0.001
- added link left_outer_finger; collision mesh filename=package://kuka_bringup/meshes/gripper/collision/robotiq_arg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 scale=0.001 0.001 0.001; visual mesh filename=package://kuka_bringup/meshes/gripper/visual/robotiq_arg2f_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 scale=0.001 0.001 0.001
- added link left_outer_knuckle; collision mesh filename=package://kuka_bringup/meshes/gripper/collision/robotiq_arg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 scale=0.001 0.001 0.001; visual mesh filename=package://kuka_bringup/meshes/gripper/visual/robotiq_arg2f_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 scale=0.001 0.001 0.001
- added link right_inner_finger; collision mesh filename=package://kuka_bringup/meshes/gripper/collision/robotiq_arg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 scale=0.001 0.001 0.001; visual mesh filename=package://kuka_bringup/meshes/gripper/visual/robotiq_arg2f_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 scale=0.001 0.001 0.001
- added link right_inner_finger_pad; collision box size=0.022 0.00635 0.0375; visual box size=0.022 0.00635 0.0375
- added link right_inner_knuckle; collision mesh filename=package://kuka_bringup/meshes/gripper/collision/robotiq_arg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 scale=0.001 0.001 0.001; visual mesh filename=package://kuka_bringup/meshes/gripper/visual/robotiq_arg2f_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 scale=0.001 0.001 0.001
- added link right_outer_finger; collision mesh filename=package://kuka_bringup/meshes/gripper/collision/robotiq_arg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 scale=0.001 0.001 0.001; visual mesh filename=package://kuka_bringup/meshes/gripper/visual/robotiq_arg2f_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 scale=0.001 0.001 0.001
- added link right_outer_knuckle; collision mesh filename=package://kuka_bringup/meshes/gripper/collision/robotiq_arg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 scale=0.001 0.001 0.001; visual mesh filename=package://kuka_bringup/meshes/gripper/visual/robotiq_arg2f_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 scale=0.001 0.001 0.001
Joints:
- added joint finger_joint: type fixed, parent gripper_base_link, child left_outer_knuckle, origin xyz=0 -0.0306011 0.054904 rpy=0 0 3.1415, axis 1 0 0, limit lower=0 upper=0.8 effort=1000 velocity=2.0
- added joint joint_a7-gripper: type fixed, parent link_7, child gripper_base_link, origin xyz=0 0 0.126 rpy=0 0 0, axis 0 0 0
- added joint left_inner_finger_joint: type fixed, parent left_outer_finger, child left_inner_finger, origin xyz=0 0.0061 0.0471 rpy=0 0 0, axis 1 0 0, limit lower=0 upper=0.8757 effort=1000 velocity=2.0
- added joint left_inner_finger_pad_joint: type fixed, parent left_inner_finger, child left_inner_finger_pad, origin xyz=0 -0.0220203446692936 0.03242 rpy=0 0 0, axis 0 0 1
- added joint left_inner_knuckle_joint: type fixed, parent gripper_base_link, child left_inner_knuckle, origin xyz=0 -0.0127 0.06142 rpy=0 0 3.1415, axis 1 0 0, limit lower=0 upper=0.8757 effort=1000 velocity=2.0
- added joint left_outer_finger_joint: type fixed, parent left_outer_knuckle, child left_outer_finger, origin xyz=0 0.0315 -0.0041 rpy=0 0 0, axis 1 0 0
- added joint right_inner_finger_joint: type fixed, parent right_outer_finger, child right_inner_finger, origin xyz=0 0.0061 0.0471 rpy=0 0 0, axis 1 0 0, limit lower=0 upper=0.8757 effort=1000 velocity=2.0
- added joint right_inner_finger_pad_joint: type fixed, parent right_inner_finger, child right_inner_finger_pad, origin xyz=0 -0.0220203446692936 0.03242 rpy=0 0 0, axis 0 0 1
- added joint right_inner_knuckle_joint: type fixed, parent gripper_base_link, child right_inner_knuckle, origin xyz=0 0.0127 0.06142 rpy=0 0 0, axis 1 0 0, limit lower=0 upper=0.8757 effort=1000 velocity=2.0
- added joint right_outer_finger_joint: type fixed, parent right_outer_knuckle, child right_outer_finger, origin xyz=0 0.0315 -0.0041 rpy=0 0 0, axis 1 0 0
- added joint right_outer_knuckle_joint: type fixed, parent gripper_base_link, child right_outer_knuckle, origin xyz=0 0.0306011 0.054904 rpy=0 0 0, axis 1 0 0, limit lower=0 upper=0.81 effort=1000 velocity=2.0
- joint joint_a1: type revolute -> fixed
- joint joint_a2: type revolute -> fixed
- joint joint_a3: type revolute -> fixed
- joint joint_a4: type revolute -> fixed
- joint joint_a5: type revolute -> fixed
- joint joint_a6: type revolute -> fixed
- joint joint_a7: type revolute -> fixed
