Commit message: added some inertia measures to urdf and sdf

File: kmr_bringup/urdf/kmr_withD435.urdf (robot description, URDF)
Before this commit: robot kmr, 40 links, 39 joints
Links:
- removed link camera_link
- added link gripper_middle_point
- link base_iiwa: mass None -> 5
- link d435_link: mass None -> 0.564; geometry collision box size=0.02505 0.090 0.025; visual mesh filename=package://kmr_bringup/meshes/sensors/visual/d435.dae
- link gripper_base_link: mass None -> 0.30915
- link left_inner_finger: mass None -> 0.00724255346165745
- link left_inner_finger_pad: mass None -> 0.019555
- link left_inner_knuckle: mass None -> 0.0110930853895903
- link left_outer_finger: mass None -> 0.0273093985570947
- link left_outer_knuckle: mass None -> 0.00684838849434396
- link link_1: mass None -> 4
- link link_2: mass None -> 4
- link link_3: mass None -> 3
- link link_4: mass None -> 2.7
- link link_5: mass None -> 1.7
- link link_6: mass None -> 1.8
- link link_7: mass None -> 0.3
- link right_inner_finger: mass None -> 0.00724255346165744
- link right_inner_finger_pad: mass None -> 0.019555
- link right_inner_knuckle: mass None -> 0.0110930853895903
- link right_outer_finger: mass None -> 0.0273093985570947
- link right_outer_knuckle: mass None -> 0.00684838849401352
Joints:
- removed joint camera_joint
- removed joint camera_joint2
- added joint d435_joint: type fixed, parent base_link_top, child camera_link, origin xyz=0.483 0.0 0.2625 rpy=0 0 0

Commit message: added inertia for box and sensors

File: kmr_bringup/urdf/kmr_withD435.urdf (robot description, URDF)
Before this commit: robot kmr, 40 links, 38 joints
Links:
- link base_link: mass 364 -> 55.04
- link base_link_middle: mass 364 -> 18.42
- link base_link_top: mass 364 -> 339.96
- link laser_B1_link: mass None -> 1.2
- link laser_B4_link: mass None -> 1.2

Commit message: renaming of nodes + making kmr drive back home when finished

File: kmr_bringup/urdf/kmr_withD435.urdf (robot description, URDF)
Before this commit: robot kmr, 40 links, 38 joints
Joints:
- added joint gripper_middle_point: type fixed, parent gripper_base_link, child gripper_middle_point, origin xyz=0 0.0 0.14 rpy=0 0 0
- joint camera_depth_joint: parent camera_link -> d435_link
- joint d435_joint: child camera_link -> d435_link

Commit message: attached camera with right frames

File: kmr_bringup/urdf/kmr_withD435.urdf (robot description, URDF)
Before this commit: robot kmr, 40 links, 39 joints
Links:
- removed link camera_depth_frame
- removed link camera_depth_optical_frame
- removed link camera_fisheye_frame
- removed link camera_fisheye_optical_frame
- removed link camera_left_ir_frame
- removed link camera_left_ir_optical_frame
- removed link camera_right_ir_frame
- removed link camera_right_ir_optical_frame
- removed link d435_link
- added link adapter; visual cylinder length=0.01 radius=0.0375
- added link camera1_depth_frame
- added link camera1_depth_optical_frame
- added link camera1_fisheye_frame
- added link camera1_fisheye_optical_frame
- added link camera1_left_ir_frame
- added link camera1_left_ir_optical_frame
- added link camera1_right_ir_frame
- added link camera1_right_ir_optical_frame
- added link d435_1_link, mass 0.564; collision box size=0.02505 0.090 0.025; visual mesh filename=package://kmr_bringup/meshes/sensors/visual/d435.dae
- added link d435_manipulator_link, mass 0.564; collision box size=0.02505 0.090 0.025; visual mesh filename=package://kmr_bringup/meshes/sensors/visual/d435.dae
Joints:
- removed joint camera_depth_joint
- removed joint camera_depth_optical_joint
- removed joint camera_fisheye_joint
- removed joint camera_fisheye_optical_joint
- removed joint camera_left_ir_joint
- removed joint camera_left_ir_optical_joint
- removed joint camera_right_ir_joint
- removed joint camera_right_ir_optical_joint
- removed joint d435_joint
- removed joint joint_a7-gripper
- added joint camera1_depth_joint: type fixed, parent d435_1_link, child camera1_depth_frame, origin xyz=0.0149 -0.0075 0.0125 rpy=0 0 0
- added joint camera1_depth_optical_joint: type fixed, parent camera1_depth_frame, child camera1_depth_optical_frame, origin xyz=0 0 0 rpy=-1.570796 0 -1.570796
- added joint camera1_fisheye_joint: type fixed, parent camera1_depth_frame, child camera1_fisheye_frame, origin xyz=0 0.040 0 rpy=0 0 0
- added joint camera1_fisheye_optical_joint: type fixed, parent camera1_fisheye_frame, child camera1_fisheye_optical_frame, origin xyz=0 0 0 rpy=-1.570796 0 -1.570796
- added joint camera1_left_ir_joint: type fixed, parent camera1_depth_frame, child camera1_left_ir_frame, origin xyz=0 -0.025 0 rpy=0 0 0
- added joint camera1_left_ir_optical_joint: type fixed, parent camera1_left_ir_frame, child camera1_left_ir_optical_frame, origin xyz=0 0 0 rpy=-1.570796 0 -1.570796
- added joint camera1_right_ir_joint: type fixed, parent camera1_depth_frame, child camera1_right_ir_frame, origin xyz=0 0.025 0 rpy=0 0 0
- added joint camera1_right_ir_optical_joint: type fixed, parent camera1_right_ir_frame, child camera1_right_ir_optical_frame, origin xyz=0 0 0 rpy=-1.570796 0 -1.570796
- added joint d435_1_joint: type fixed, parent base_link_top, child d435_1_link, origin xyz=0.483 0.0 0.2625 rpy=0 0 0
- added joint d435_manipulator_joint: type fixed, parent adapter, child d435_manipulator_link, origin xyz=-0.0375 0.0 0.0 rpy=0 -1.570796 0
- added joint joint_a7-adapter: type fixed, parent link_7, child adapter, origin xyz=0 0 0.126 rpy=0 0 0, axis 0 0 0
- added joint joint_adapter-gripper: type fixed, parent adapter, child gripper_base_link, origin xyz=0 0 0.005 rpy=0 0 0, axis 0 0 0

Commit message: added two more cameras to base

File: kmr_bringup/urdf/kmr_withD435.urdf (robot description, URDF)
Before this commit: robot kmr, 42 links, 41 joints
Links:
- removed link camera1_depth_frame
- removed link camera1_depth_optical_frame
- removed link camera1_fisheye_frame
- removed link camera1_fisheye_optical_frame
- removed link camera1_left_ir_frame
- removed link camera1_left_ir_optical_frame
- removed link camera1_right_ir_frame
- removed link camera1_right_ir_optical_frame
- removed link d435_1_link
- added link d435_base_front_depth_frame
- added link d435_base_front_depth_optical_frame
- added link d435_base_front_fisheye_frame
- added link d435_base_front_fisheye_optical_frame
- added link d435_base_front_left_ir_frame
- added link d435_base_front_left_ir_optical_frame
- added link d435_base_front_link, mass 0.564; collision box size=0.02505 0.090 0.025; visual mesh filename=package://kmr_bringup/meshes/sensors/visual/d435.dae
- added link d435_base_front_right_ir_frame
- added link d435_base_front_right_ir_optical_frame
- added link d435_base_left_link, mass 0.564; collision box size=0.02505 0.090 0.025; visual mesh filename=package://kmr_bringup/meshes/sensors/visual/d435.dae
- added link d435_base_right_link, mass 0.564; collision box size=0.02505 0.090 0.025; visual mesh filename=package://kmr_bringup/meshes/sensors/visual/d435.dae
- added link metall_plate_left_link; collision box size=0.2 0.04 0.01; visual box size=0.2 0.04 0.01
- added link metall_plate_right_link; collision box size=0.2 0.04 0.01; visual box size=0.2 0.04 0.01
Joints:
- removed joint camera1_depth_joint
- removed joint camera1_depth_optical_joint
- removed joint camera1_fisheye_joint
- removed joint camera1_fisheye_optical_joint
- removed joint camera1_left_ir_joint
- removed joint camera1_left_ir_optical_joint
- removed joint camera1_right_ir_joint
- removed joint camera1_right_ir_optical_joint
- removed joint d435_1_joint
- added joint d435_base_front_depth_joint: type fixed, parent d435_base_front_link, child d435_base_front_depth_frame, origin xyz=0.0149 -0.0075 0.0125 rpy=0 0 0
- added joint d435_base_front_depth_optical_joint: type fixed, parent d435_base_front_depth_frame, child d435_base_front_depth_optical_frame, origin xyz=0 0 0 rpy=-1.570796 0 -1.570796
- added joint d435_base_front_fisheye_joint: type fixed, parent d435_base_front_depth_frame, child d435_base_front_fisheye_frame, origin xyz=0 0.040 0 rpy=0 0 0
- added joint d435_base_front_fisheye_optical_joint: type fixed, parent d435_base_front_fisheye_frame, child d435_base_front_fisheye_optical_frame, origin xyz=0 0 0 rpy=-1.570796 0 -1.570796
- added joint d435_base_front_joint: type fixed, parent base_link_top, child d435_base_front_link, origin xyz=0.52 0.0 0.2625 rpy=0 0 0
- added joint d435_base_front_left_ir_joint: type fixed, parent d435_base_front_depth_frame, child d435_base_front_left_ir_frame, origin xyz=0 -0.025 0 rpy=0 0 0
- added joint d435_base_front_left_ir_optical_joint: type fixed, parent d435_base_front_left_ir_frame, child d435_base_front_left_ir_optical_frame, origin xyz=0 0 0 rpy=-1.570796 0 -1.570796
- added joint d435_base_front_right_ir_joint: type fixed, parent d435_base_front_depth_frame, child d435_base_front_right_ir_frame, origin xyz=0 0.025 0 rpy=0 0 0
- added joint d435_base_front_right_ir_optical_joint: type fixed, parent d435_base_front_right_ir_frame, child d435_base_front_right_ir_optical_frame, origin xyz=0 0 0 rpy=-1.570796 0 -1.570796
- added joint d435_base_left_joint: type fixed, parent metall_plate_left_link, child d435_base_left_link, origin xyz=0.0 0.0 0.005 rpy=0 0.0 1.570796
- added joint d435_base_right_joint: type fixed, parent metall_plate_right_link, child d435_base_right_link, origin xyz=0.0 0.0 0.005 rpy=0 0 -1.570796
- added joint metall_plate_left_joint: type fixed, parent base_link_top, child metall_plate_left_link, origin xyz=-0.08 0.28 0.2675 rpy=0 0 0
- added joint metall_plate_right_joint: type fixed, parent base_link_top, child metall_plate_right_link, origin xyz=-0.08 -0.28 0.2675 rpy=0 0 0

Commit message: tf frames of d435 cameras at base fixed - pointcloud publishing correct

File: kmr_bringup/urdf/kmr_withD435.urdf (robot description, URDF)
Before this commit: robot kmr, 46 links, 45 joints
Links:
- removed link d435_base_front_depth_frame
- removed link d435_base_front_depth_optical_frame
- removed link d435_base_front_fisheye_frame
- removed link d435_base_front_fisheye_optical_frame
- removed link d435_base_front_left_ir_frame
- removed link d435_base_front_left_ir_optical_frame
- removed link d435_base_front_right_ir_frame
- removed link d435_base_front_right_ir_optical_frame
Joints:
- removed joint d435_base_front_depth_joint
- removed joint d435_base_front_depth_optical_joint
- removed joint d435_base_front_fisheye_joint
- removed joint d435_base_front_fisheye_optical_joint
- removed joint d435_base_front_left_ir_joint
- removed joint d435_base_front_left_ir_optical_joint
- removed joint d435_base_front_right_ir_joint
- removed joint d435_base_front_right_ir_optical_joint
- joint d435_base_front_joint: origin xyz=0.52 0.0 0.2625 rpy=0 0 0 -> xyz=0.52 0.0 0.2625 rpy=-1.570796 0 -1.570796 
- joint d435_base_left_joint: origin xyz=0.0 0.0 0.005 rpy=0 0.0 1.570796 -> xyz=0.0 0.0 0.005 rpy=-1.570796 0 0
- joint d435_base_right_joint: origin xyz=0.0 0.0 0.005 rpy=0 0 -1.570796 -> xyz=0.0 0.0 0.005 rpy=-1.570796 0 3.1415

Commit message: working on navigation with BT

File: kmr_bringup/urdf/kmr_withD435.urdf (robot description, URDF)
Before this commit: robot kmr, 38 links, 37 joints
Links:
- added link d435_base_front_depth_frame
Joints:
- added joint d435_base_front_depth_joint: type fixed, parent d435_base_front_link, child d435_base_front_depth_frame, origin xyz=0.0149 -0.0075 0.0125 rpy=0 0 0
- joint joint_a1: type revolute -> fixed
- joint joint_a2: type revolute -> fixed
- joint joint_a3: type revolute -> fixed
- joint joint_a4: type revolute -> fixed
- joint joint_a5: type revolute -> fixed
- joint joint_a6: type revolute -> fixed
- joint joint_a7: type revolute -> fixed
