Commit message: nuc files and cartographer tuning

File: kmr_bringup/urdf/kmriiwa.urdf (robot description, URDF)
Before this commit: robot kmr, 46 links, 45 joints
Links:
- removed link d435_base_front_fisheye_frame
- removed link d435_base_front_fisheye_optical_frame
- removed link d435_base_front_left_ir_frame
- removed link d435_base_front_left_ir_optical_frame
- removed link d435_base_front_right_ir_frame
- removed link d435_base_front_right_ir_optical_frame
Joints:
- removed joint d435_base_front_fisheye_joint
- removed joint d435_base_front_fisheye_optical_joint
- removed joint d435_base_front_left_ir_joint
- removed joint d435_base_front_left_ir_optical_joint
- removed joint d435_base_front_right_ir_joint
- removed joint d435_base_front_right_ir_optical_joint

Commit message: fixed size of adapter

File: kmr_bringup/urdf/kmriiwa.urdf (robot description, URDF)
Before this commit: robot kmr, 40 links, 39 joints
Links:
- removed link tool0
- link adapter: geometry visual cylinder length=0.035 radius=0.0375
Joints:
- removed joint joint_a7-tool0
- joint joint_a1: type revolute -> fixed
- joint joint_a2: type revolute -> fixed
- joint joint_a3: type revolute -> fixed
- joint joint_a4: type revolute -> fixed
- joint joint_a5: type revolute -> fixed
- joint joint_a6: type revolute -> fixed
- joint joint_a7: type revolute -> fixed
- joint joint_a7-adapter: origin xyz=0 0 0.126 rpy=0 0 0 -> xyz=0 0 0.1365 rpy=0 0 0
- joint joint_adapter-gripper: origin xyz=0 0 0.005 rpy=0 0 0 -> xyz=0 0 0.0175 rpy=0 0 0

Commit message: attached camera to manipulator

File: kmr_bringup/urdf/kmriiwa.urdf (robot description, URDF)
Before this commit: robot kmr, 39 links, 38 joints
Links:
- added link kamerafeste1; visual box size=0.01 0.015 0.01
- added link kamerafeste2; visual box size=0.01 0.015 0.02
Joints:
- added joint joint_adapter-feste1: type fixed, parent adapter, child kamerafeste1, origin xyz=-0.0425 0 0.0125 rpy=0 0 0, axis 0 0 0
- added joint joint_adapter-feste2: type fixed, parent kamerafeste1, child kamerafeste2, origin xyz=-0.01 0 0.005 rpy=0 0 0, axis 0 0 0
- joint d435_manipulator_joint: origin xyz=-0.0375 0.0 0.0 rpy=0 -1.570796 0 -> xyz=-0.005 0.0 0.005 rpy=0 -1.570796 0; parent adapter -> kamerafeste2

Commit message: added gripper adapter link

File: kmr_bringup/urdf/kmriiwa.urdf (robot description, URDF)
Before this commit: robot kmr, 41 links, 40 joints
Links:
- added link d435_manipulator_depth_frame
- added link d435_manipulator_depth_optical_frame
- added link gripper-adapter; visual cylinder length=0.016 radius=0.0375
Joints:
- removed joint joint_adapter-gripper
- added joint d435_manipulator_depth_joint: type fixed, parent d435_manipulator_link, child d435_manipulator_depth_frame, origin xyz=0.0149 -0.0075 0.0125 rpy=0 0 0
- added joint d435_manipulator_depth_optical_joint: type fixed, parent d435_manipulator_depth_frame, child d435_manipulator_depth_optical_frame, origin xyz=0 0 0 rpy=-1.570796 0 -1.570796
- added joint joint_adapter-gripperadapter: type fixed, parent adapter, child gripper-adapter, origin xyz=0 0 0.0255 rpy=0 0 0, axis 0 0 0
- added joint joint_gripperadapter-gripper: type fixed, parent gripper-adapter, child gripper_base_link, origin xyz=0 0 0.008 rpy=0 0 0, axis 0 0 0
- joint gripper_middle_point: origin xyz=0 0.0 0.14 rpy=0 0 0 -> xyz=0 0.0 0.144 rpy=0 0 0
- joint joint_a1: type fixed -> revolute
- joint joint_a2: type fixed -> revolute
- joint joint_a3: type fixed -> revolute
- joint joint_a4: type fixed -> revolute
- joint joint_a5: type fixed -> revolute
- joint joint_a6: type fixed -> revolute
- joint joint_a7: type fixed -> revolute
- joint joint_a7-adapter: origin xyz=0 0 0.1365 rpy=0 0 0 -> xyz=0 0 0.1365 rpy=0 0 -0.785398

File: kmr_bringup/urdf/kmriiwa_withcameraframes.urdf (robot description, URDF)
Before this commit: robot kmr, 46 links, 45 joints
Links:
- removed link camera1_color_optical_frame_link
- removed link camera1_depth_optical_frame_link
- added link d435_base_front_color_optical_frame_link
- added link d435_base_front_depth_optical_frame_link
Joints:
- joint bf: origin xyz=0 0 0 rpy=0 0 0.0775 -> xyz=0 0 0.0775 rpy=0 0 0
- joint d435_base_front_color_joint: child camera1_color_optical_frame_link -> d435_base_front_color_optical_frame_link
- joint d435_base_front_depth_joint: child camera1_depth_optical_frame_link -> d435_base_front_depth_optical_frame_link

Commit message: licence and remove comments

File: kmr_bringup/urdf/kmriiwa.urdf (robot description, URDF)
Before this commit: robot kmr, 44 links, 43 joints
Joints:
- joint bf: origin xyz=0 0 0 rpy=0 0 0.0775 -> xyz=0 0 0.0775 rpy=0 0 0.0
